Commit message: Add Isaac Sim synthetic data generation for CV training
New goal for this layer, per direction: use the digital twin not just to
mirror the real rig, but to mass-produce labeled training data for the
stone-detection CV system from the rig's own simulated camera.

  - urdf: camera_link, a fixed mount point at the flexion tip (placeholder
    offset, documented as such).
  - ros2/isaac/_isaac_common.py: pulled the URDF-import code out of
    load_rig.py so generate_training_data.py doesn't duplicate it.
  - ros2/isaac/generate_training_data.py: Replicator-based synthetic data
    generator -- placeholder calyx/ureter anatomy, randomized stones
    (count/size/color/pose), randomized lighting and tissue tint, an
    optional --dynamic mode where stones drift under rigid-body physics at
    the clinical 1-10 mm/s rate, auto-labeled RGB + segmentation mask +
    depth + bounding box output via Isaac's BasicWriter.
  - ros2/isaac/CAMERA-SPECS.md: the exact real-world measurements needed
    (camera intrinsics, mount offset, lighting spec, anatomy/stone
    reference imagery) to turn the current placeholders into a dataset
    that actually transfers to the real feed, in priority order.

Same caveat as the rest of ros2/isaac, stated plainly in both the script's
docstring and the READMEs: written against NVIDIA's documented Isaac Sim
6.x Replicator API, not run against a real install -- none was available
here.

Co-Authored-By: Claude Sonnet 5 <noreply@anthropic.com>
Claude-Session: https://claude.ai/code/session_01VUhBeVcdabfg2M1WayJYJe

File: ros2/katzlab_bridge/urdf/ureteroscope.urdf (robot description, URDF)
Before this commit: robot ureteroscope, 4 links, 3 joints
Links:
- added link camera_link; visual box size=0.002 0.002 0.002
Joints:
- added joint camera_joint: type fixed, parent flexion_link, child camera_link, origin xyz=0.04 0 0 rpy=0 0 0
